File: Projects/Analog_Inputs/Analog_Input.sch (EAGLE design)
At the start: 35 parts, among them U1 LM324, U2 ACS70331EESATR-005U3, U3 DIP-GAS-MQ-9(6P-D19MM), U4 NA555DR

Commit message: Most recent batch of new components
Parts:
- removed R4, R5: TBD, ngspice-simulation:R
- C8: value TBD -> 10uF
- C9: value TBD -> 1uF
- R1: value TBD -> 680k
- R2: value TBD -> 50k
- R3, R6, R7: value TBD -> 1M
Connections:
- removed net N$16: C8.2, R6.1, U4.THRES
- net GND: now also R3.2; no longer R2.1, R4.2
- net N$11: now also R1.2, R2.1, U1G$4.NON-INVERTING_INPUT4; no longer R3.1, R4.1, U1G$3.INVERTING_INPUT3
- net N$14: now also R3.1, U1G$3.INVERTING_INPUT3; no longer R1.1, U1G$4.NON-INVERTING_INPUT4
- net THRESH_NET: now also C8.2, R6.1, U4.THRES
- net TO_DISC_IN: no longer R5.2
- net VDD: now also R1.1; no longer R1.2, R3.2, R5.1
Other:
- moved on the sheet: R1, R2, R3

Commit message: Updated Schematics
Parts:
- removed R17, R18, R8: TBD, ngspice-simulation:R
- removed U$2: MULTIPLEXER_SN74, Multiplexer_SN74HC153PWR:MULTIPLEXER_SN74
- added R4: 10k, ngspice-simulation:R
- added U$3: MQ_7, MQ_7:MQ_7
- C4: value 0.1uF -> 100uF
- U3: value DIP-GAS-MQ-9(6P-D19MM) -> 74HC4051PW,118; device DIP-GAS-MQ-9_6P-D19MM_:DIP-GAS-MQ-9(6P-D19MM) -> 74HC4051PW_118:74HC4051PW,118
Connections:
- removed net N$10: C4.1, R10.1
- removed net N$13: U1G$1.OUTPUT1, U1G$3.NON-INVERTING_INPUT3, U1G$4.INVERTING_INPUT4
- removed net N$20: R17.2, R8.1, U3.H@1
- removed net VDD: C1.2, R1.1, R11.2, R17.1, R18.1, R6.2, R7.2, U$1.+5V, U$2.VCC, U1G$1.VCC+, U2.IP+, U2.IP-, U2.VCC, U4.RESET, U4.VCC
- new net 3V3_BRD: R1.1, U2.IP-, U2.VCC, U3.S2, U3.VCC, U3.VEE
- new net 3V3_REG: U2.IP+
- new net 5V: C1.2, R11.2, R6.2, R7.2, U$1.+5V, U$3.VCC, U1G$1.VCC+, U4.RESET, U4.VCC
- new net D1: U3.S0
- new net D2: U3.S1
- new net N$16: U$3.A0, U3.Y1
- net ANALOG_IN: now also U3.Z; no longer U$2.1Y
- net GND: now also C4.1, R10.1, R4.1, U$3.GND, U3.GND; no longer R8.2, U$2.GND, U3.B0, U3.B1, U3.H@2
- net N$21: now also R4.2, U3.~E; no longer R18.2, U$2.1C2, U3.A0, U3.A1
- net N$7: now also U3.Y0; no longer U$2.1C3
- net N$8: now also U1G$1.OUTPUT1, U1G$3.NON-INVERTING_INPUT3, U1G$4.INVERTING_INPUT4
