File: Projects/ESP32/ESP32.sch (EAGLE design)
At the start: 28 parts, among them J1 10118193-0001LF, Q1 SS8050-G, Q2 SS8050-G, SW1 OS102011MS2QN1, SW2 OS102011MS2QN1, U1 FT260Q-T, U2 MIC5387-SGFYMT-TR, U3 ESP32-WROOM-32E_(16MB)

Commit message: Updated Schematics
Parts:
- R7: value 2k -> 2.2k
- R8: value 10 -> 10k
Connections:
- net 3V3_REG renamed 3V3_BRD
- removed net VCC: C1.1, C3.1, D1.K, R3.2, R7.1, R8.1, U1.VCCIN, U2.OUT1, U2.VIN
- new net 3V3_USB: C3.1, R3.2, R7.1, U2.OUT1
- new net 5V_EXT: C1.1, D1.K, R8.1, U1.VCCIN, U2.VIN
- net GND: now also U2.EN2/3
