File: Projects/Full_Schematic/Full_Schematic.sch (EAGLE design)
At the start: 82 parts, among them J1 10118193-0001LF, Q1 SS8050-G, Q2 SS8050-G, SW1 OS102011MS2QN1, SW2 OS102011MS2QN1, U1 LM324, U10 SC189ZSKTRT, U2 ACS70331EESATR-005U3, U3 74HC4051PW,118, U4 NA555DR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

Commit message: Update Full_Schematic.sch
Parts:
- removed C16: 22uF, ngspice-simulation:C
- removed D2: BAT760-7, BAT760-7:BAT760-7
Connections:
- removed net 5V_BRD: D3.K
- removed net ANALOG_IN: U3.Z
- removed net ESP_SCL: R63.1, R64.2, U8.SCL, U9.SCL
- removed net ESP_SDA: R62.1, R65.2, U8.SDA, U9.SDA
- removed net N$10: U2.VCC
- removed net N$40: U7.IO17
- removed net N$41: U7.IO18
- removed net N$43: U7.IO21
- removed net N$44: U7.IO22
- removed net N$49: U7.IO32
- removed net N$59: D2.K
- new net 3V3_SENSE_IN: D4.K, D5.K, U2.IP+, U2.VCC
- new net ADC_IN: U3.Z, U7.IO32
- new net I2C_SCL: R63.1, R64.2, U7.IO22, U8.SCL, U9.SCL
- new net I2C_SDA: R62.1, R65.2, U7.IO21, U8.SDA, U9.SDA
- net 3V3_BRD: now also C5.2; no longer C16.1, D4.K, D5.K
- net 3V3_REG: no longer D2.A, U2.IP+
- net 5V: now also D3.K
- net D1: now also U7.IO17
- net D2: now also U7.IO18
- net GND: now also C5.1; no longer C16.2
Other:
- note added: "3V3_BRD is the power source for everything on the board. It is the regulated input for both the USB and battery supply"
- moved on the sheet: C5

Commit message: Final revision of the Full Schematic, haven't updated in a while since I was soloing this one.
Parts:
- removed CR1, CR2: 1N4148WX-TP, 1n4148WX-TP_Diode:1N4148WX-TP
- removed R36, R37, R38, R47: 10k, rcl:R-US_R0402
- removed R46: 73k, rcl:R-US_R0402
- removed R56: 680k, rcl:R-US_R0402
- removed R57: 50k, rcl:R-US_R0402
- removed R58, R59: 1M, rcl:R-US_R0402
- removed R64, R65: 2.2k, rcl:R-US_R0402
- added C7: 1uF, rcl:C-EUC0603
- added J5: 691137710002, 691137710002:691137710002
- added J6, J7: 826629-8, 826629-8:826629-8
- added R3: 2.2k, rcl:R-US_R0402
- added U$5: 2PIN_HEADER, 2PIN_HEADER:2PIN_HEADER
- added U11, U12, U13: ESD5Z5.0T1G, Circuit_protection_diode:ESD5Z5.0T1G
- C4: value 22uF -> 1uF
- U$1: value HB100 -> 2PIN_HEADER; device HB100_Doppler:HB100 -> 2PIN_HEADER:2PIN_HEADER
- U$2: value POWER_CONN -> 2PIN_HEADER; device PWR_IN:POWER_CONN -> 2PIN_HEADER:2PIN_HEADER
- renumbered C14 to C4
Connections:
- removed net N$1: C2.2, R50.2, U$1.IF
- removed net N$11: R56.1, R57.2, U1G$4.NON-INVERTING_INPUT4
- removed net N$15: CR1.1, U1G$3.OUTPUT3
- removed net N$17: CR1.2, CR2.2, R59.1, U4.TRIG
- removed net N$18: CR2.1, U1G$4.OUTPUT4
- removed net N$36: U7.IO13
- removed net N$48: U7.IO27
- removed net N$58: R46.1, R47.2, U$4.FB
- removed net N$61: R57.1, R58.2, U1G$3.INVERTING_INPUT3
- removed net N$8 (its old number): C22.2, R54.2, U1G$1.OUTPUT1, U1G$3.NON-INVERTING_INPUT3, U1G$4.INVERTING_INPUT4
- removed net RXD: R36.1, U5.DIO3
- removed net TO_DISC_IN: U4.OUT
- removed net TXD: R37.1, U5.DIO4
- new net 555_OUT: J6.P5, U4.OUT, U7.IO13
- new net D3: U3.S2, U7.IO27
- new net N$10: C27.1, R40.1, SW1.2
- new net N$2: C26.1, R41.1, SW2.2
- net 3V3_BRD: now also J6.P6, U$4.FB, U8.VDDH; no longer R56.2, R64.1, R65.1, U3.S2
- net 3V3_EXT: now also J5.1; no longer U$2.3V3_RAW
- net 3V3_REG: now also J7.P5
- net 3V3_USB: now also C7.2, J7.P4, R3.2
- net 5V: now also J6.P8, U$2.1, U$2.2; no longer R59.2, U$1.+5V
- net 5V1: no longer R46.2
- net ADC_IN: now also J6.P7
- net D1: now also U7.IO14; no longer U7.IO17
- net D2: now also U7.IO12; no longer U7.IO18
- net DTRN: now also J7.P7
- net EN: now also J7.P6, R41.2; no longer C26.1, R41.1, SW2.2
- net GND: now also C7.1, J5.2, U$5.1, U$5.2, U11.ANODE, U12.ANODE, U13.ANODE, U5.DCNF0, U5.DCNF1, U6.7; no longer R38.2, R47.1, R58.1, U$1.GND, U$2.GND
- net I2C_SCL: now also J6.P3; no longer R64.2
- net I2C_SDA: now also J6.P1; no longer R65.2
- net IO0: now also J7.P3, R40.2; no longer C27.1, R40.1, SW1.2
- net N$16: now also J6.P2
- net N$20: now also U13.CATHODE
- net N$22: now also U11.CATHODE
- net N$23: now also U12.CATHODE
- net N$29: now also C2.2, R50.2, U$1.1, U$1.2; no longer R41.2
- net N$30: now also R3.1, U5.STEST_RSTN; no longer R40.2
- net N$35: now also U7.IO17; no longer U7.IO12
- net N$37: now also U7.IO18; no longer U7.IO14
- net N$6: now also U1G$1.NON-INVERTING_INPUT1; no longer U1G$1.INVERTING_INPUT1
- net N$7: now also J6.P4
- net N$9: now also U1G$1.INVERTING_INPUT1; no longer U1G$1.NON-INVERTING_INPUT1
- net RTSN: now also J7.P8
- net RXD0: now also J7.P2, U5.DIO4; no longer R37.2
- net SUSPENDN: no longer R38.1
- net THRESH_NET: now also C22.2, R54.2, U1G$1.OUTPUT1, U4.TRIG
- net TXD0: now also J7.P1, U5.DIO3; no longer R36.2
Other:
- note added: "10k resistor, dnp"
- note added: "Added a resistor that the archetype doesn't have, didn't want to short the IO0 and EN pins to GND"
- note added: "Current time value is approximately ten seconds, needs to be documented somewhere more important than this schematic"
- note added: "Formerly weird pads to solder to, now using a terminal block"
- note added: "I didn't want the current sensor's current to be recorded, so the 3V3_SENSE_IN is used to power this device"
- note added: "Somewhat confusing, some of the design from the ESP32 schematic is used here with the regulator, but it's verified. Probably going to move the ESP32 stuff to the ESP32 area in the future but leaving it for now"
- note added: "Test headers, 1x8 2.54mm pitch, so standard test header"
- note added: "This section is flipped from the archetype shoen by ESPRESSIF reference uses rts and dtr, I have Rtsn and DTRN so the outputs are flipped"
- note added: "Using the 0333 instead of the 033, so FB should connect to VIN as the output can only be 5V Datasheet at https://www.digikey.gr/en/products/detail/texas-instruments/TPS610333DRLR/22106777"
- note added: "https://dl.espressif.com/dl/schematics/esp32_devkitc_v4-sch.pdf for a very large majority of thr design in this PCB"
- note added: "https://semtech.my.salesforce.com/sfc/p/#E0000000JelG/a/44000000MDZF/Kz5ycNi9I5Dzzg5AzBOB4W0TtqtKUtMf03CWPRt6CLQ"
- note removed: "Need RC values to hold output high for a long time, I'm currently thinking ten seconds but that's TBD"
- note removed: "Need to re-check resistor values, especially the 100k resistor. Thinking of checking in with a professor about the configuration for this part."
- note removed: "Resistor values need chosen to hold output default high, input range for high voltage is TBD"
- moved on the sheet: C1, C12, C2, C21, C22, C23, C24, C25, C3, C8, R40, R41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
